Commit message: Update hokuyo

File: p3dx_description/urdf/p3dx/pioneer3dx.xacro (robot description, xacro)
@@ -1,4 +1,5 @@
 <?xml version="1.0"?>
 <robot xmlns:xacro="http://wiki.ros.org/xacro" name="pioneer3dx">
+  <xacro:property name="M_PI" value="3.1415926535897931" />
   <!-- Import Rviz colors -->
   <xacro:include filename="$(find p3dx_description)/urdf/materials.xacro" />
@@ -8,6 +9,6 @@
   <!-- Hokuyo UTM-30LX -->
   <xacro:include filename="$(find p3dx_description)/urdf/sensors/hokuyo_utm30lx.urdf.xacro" />
-  <xacro:element xacro:name="sensor_hokuyo_utm30lx" prefix="hokuyo_utm30lx" parent="chassis" meshes="package://p3dx_description/meshes/sensors" min_angle="-2.3562" max_angle="2.3562" >
+  <xacro:sensor_hokuyo_utm30lx prefix="hokuyo_utm30lx" parent="chassis" meshes="package://p3dx_description/meshes/sensors" min_angle="${-135.0*M_PI/180.0}" max_angle="${135.0*M_PI/180.0}" >
     <origin xyz="0.12 0 0.23" rpy="0 0 0"/>
-  </xacro:element>
+  </xacro:sensor_hokuyo_utm30lx>
 </robot>

File: p3dx_description/urdf/sensors/hokuyo_utm30lx.urdf.xacro (robot description, xacro)
@@ -2,5 +2,6 @@
 <robot name="sensor_hokuyo_utm30lx"
   xmlns:xacro="http://wiki.ros.org/xacro">
-  <xacro:macro name="sensor_hokuyo_utm30lx" params="prefix parent meshes prefix_topic:='' *origin min_angle:=-2.356194 max_angle:=2.356194 gpu:=^|true">
+  <xacro:property name="M_PI" value="3.1415926535897931" />
+  <xacro:macro name="sensor_hokuyo_utm30lx" params="prefix parent meshes prefix_topic:='' *origin min_angle:='${-135.0*M_PI/180.0}' max_angle:='${135.0*M_PI/180.0}' gpu:=^|true">
     <joint name="${prefix}_base_joint" type="fixed">
       <!-- FRONT MOUNT  -->
@@ -33,46 +34,6 @@
     </joint>
     <!-- Hokuyo sensor for simulation -->
-    <sensor_hokuyo_utm_gazebo/>
-  </xacro:macro>
-  <xacro:macro name="sensor_hokuyo_utm_gazebo">
-    <gazebo reference="${prefix}_link">
-      <xacro:if value="${gpu}">
-        <xacro:property name="ray_type" value="gpu_ray" />
-        <xacro:property name="plugin_lib" value="libgazebo_ros_gpu_laser.so" />
-      </xacro:if>
-      <xacro:unless value="${gpu}">
-        <xacro:property name="ray_type" value="ray" />
-        <xacro:property name="plugin_lib" value="libgazebo_ros_laser.so" />
-      </xacro:unless>
-      <sensor type="${ray_type}" name="${prefix}_sensor">
-        <pose>0 0 0 0 0 0</pose>
-        <visualize>false</visualize>
-        <update_rate>30</update_rate>
-        <ray>
-          <scan>
-            <horizontal>
-              <samples>1081</samples>
-              <resolution>1</resolution>
-              <min_angle>${min_angle}</min_angle>
-              <max_angle>${max_angle}</max_angle>
-            </horizontal>
-          </scan>
-          <range>
-            <min>0.10</min>
-            <max>30.0</max>
-            <resolution>0.01</resolution>
-          </range>
-          <noise>
-            <type>gaussian</type>
-            <mean>0.0</mean>
-            <stddev>0.01</stddev>
-          </noise>
-        </ray>
-        <plugin name="${prefix}_controller" filename="${plugin_lib}">
-          <topicName>${prefix_topic}/scan</topicName>
-          <frameName>/${prefix}_link</frameName>
-        </plugin>
-      </sensor>
-    </gazebo>
+    <xacro:include filename="$(find p3dx_description)/urdf/sensors/sensor_hokuyo_utm_gazebo.urdf.xacro" />
+    <xacro:sensor_hokuyo_utm_gazebo prefix="${prefix}" prefix_topic="${prefix_topic}" min_angle="${min_angle}" max_angle="${max_angle}" gpu="${gpu}"/>
   </xacro:macro>
 </robot>
