Commit message: Update hokuyo

File: p3dx_description/urdf/sensors/hokuyo_utm30lx.urdf.xacro (robot description, xacro)
@@ -34,6 +34,46 @@
     </joint>
     <!-- Hokuyo sensor for simulation -->
-    <xacro:include filename="$(find p3dx_description)/urdf/sensors/sensor_hokuyo_utm_gazebo.urdf.xacro" />
     <xacro:sensor_hokuyo_utm_gazebo prefix="${prefix}" prefix_topic="${prefix_topic}" min_angle="${min_angle}" max_angle="${max_angle}" gpu="${gpu}"/>
   </xacro:macro>
+  <xacro:macro name="sensor_hokuyo_utm_gazebo" params="prefix prefix_topic:='' min_angle:='${-135.0*M_PI/180.0}' max_angle:='${135.0*M_PI/180.0}' gpu:=^|true">
+    <gazebo reference="${prefix}_link">
+      <xacro:if value="${gpu}">
+        <xacro:property name="ray_type" value="gpu_ray" />
+        <xacro:property name="plugin_lib" value="libgazebo_ros_gpu_laser.so" />
+      </xacro:if>
+      <xacro:unless value="${gpu}">
+        <xacro:property name="ray_type" value="ray" />
+        <xacro:property name="plugin_lib" value="libgazebo_ros_laser.so" />
+      </xacro:unless>
+      <sensor type="${ray_type}" name="${prefix}_sensor">
+        <pose>0 0 0 0 0 0</pose>
+        <visualize>false</visualize>
+        <update_rate>30</update_rate>
+        <ray>
+          <scan>
+            <horizontal>
+              <samples>1081</samples>
+              <resolution>1</resolution>
+              <min_angle>${min_angle}</min_angle>
+              <max_angle>${max_angle}</max_angle>
+            </horizontal>
+          </scan>
+          <range>
+            <min>0.10</min>
+            <max>30.0</max>
+            <resolution>0.01</resolution>
+          </range>
+          <noise>
+            <type>gaussian</type>
+            <mean>0.0</mean>
+            <stddev>0.01</stddev>
+          </noise>
+        </ray>
+        <plugin name="${prefix}_controller" filename="${plugin_lib}">
+          <topicName>${prefix_topic}/scan</topicName>
+          <frameName>/${prefix}_link</frameName>
+        </plugin>
+      </sensor>
+    </gazebo>
+  </xacro:macro>
 </robot>

Commit message: Update Hokuyo

File: p3dx_description/urdf/sensors/hokuyo_utm30lx.urdf.xacro (robot description, xacro)
@@ -3,5 +3,5 @@
   xmlns:xacro="http://wiki.ros.org/xacro">
   <xacro:property name="M_PI" value="3.1415926535897931" />
-  <xacro:macro name="sensor_hokuyo_utm30lx" params="prefix parent meshes prefix_topic:='' *origin min_angle:='${-135.0*M_PI/180.0}' max_angle:='${135.0*M_PI/180.0}' gpu:=^|true">
+  <xacro:macro name="sensor_hokuyo_utm30lx" params="prefix parent meshes prefix_topic:='' *origin min_angle:='${-135.0*M_PI/180.0}' max_angle:='${135.0*M_PI/180.0}' gpu:=false">
     <joint name="${prefix}_base_joint" type="fixed">
       <!-- FRONT MOUNT  -->
@@ -36,43 +36,68 @@
     <xacro:sensor_hokuyo_utm_gazebo prefix="${prefix}" prefix_topic="${prefix_topic}" min_angle="${min_angle}" max_angle="${max_angle}" gpu="${gpu}"/>
   </xacro:macro>
-  <xacro:macro name="sensor_hokuyo_utm_gazebo" params="prefix prefix_topic:='' min_angle:='${-135.0*M_PI/180.0}' max_angle:='${135.0*M_PI/180.0}' gpu:=^|true">
+  <xacro:macro name="sensor_hokuyo_utm_gazebo" params="prefix prefix_topic:='' min_angle:='${-135.0*M_PI/180.0}' max_angle:='${135.0*M_PI/180.0}' gpu:=false">
     <gazebo reference="${prefix}_link">
       <xacro:if value="${gpu}">
-        <xacro:property name="ray_type" value="gpu_ray" />
-        <xacro:property name="plugin_lib" value="libgazebo_ros_gpu_laser.so" />
+        <sensor type="gpu_ray" name="${prefix}_sensor">
+          <pose>0 0 0 0 0 0</pose>
+          <visualize>false</visualize>
+          <update_rate>30</update_rate>
+          <ray>
+            <scan>
+              <horizontal>
+                <samples>1081</samples>
+                <resolution>1</resolution>
+                <min_angle>${min_angle}</min_angle>
+                <max_angle>${max_angle}</max_angle>
+              </horizontal>
+            </scan>
+            <range>
+              <min>0.10</min>
+              <max>30.0</max>
+              <resolution>0.01</resolution>
+            </range>
+            <noise>
+              <type>gaussian</type>
+              <mean>0.0</mean>
+              <stddev>0.001</stddev>
+            </noise>
+          </ray>
+          <plugin name="${prefix}_controller" filename="libgazebo_ros_gpu_laser.so">
+            <topicName>${prefix_topic}/scan</topicName>
+            <frameName>/${prefix}_link</frameName>
+          </plugin>
+        </sensor>
       </xacro:if>
       <xacro:unless value="${gpu}">
-        <xacro:property name="ray_type" value="ray" />
-        <xacro:property name="plugin_lib" value="libgazebo_ros_laser.so" />
+        <sensor type="ray" name="${prefix}_sensor">
+          <pose>0 0 0 0 0 0</pose>
+          <visualize>false</visualize>
+          <update_rate>30</update_rate>
+          <ray>
+            <scan>
+              <horizontal>
+                <samples>1081</samples>
+                <resolution>1</resolution>
+                <min_angle>${min_angle}</min_angle>
+                <max_angle>${max_angle}</max_angle>
+              </horizontal>
+            </scan>
+            <range>
+              <min>0.10</min>
+              <max>30.0</max>
+              <resolution>0.01</resolution>
+            </range>
+            <noise>
+              <type>gaussian</type>
+              <mean>0.0</mean>
+              <stddev>0.001</stddev>
+            </noise>
+          </ray>
+          <plugin name="${prefix}_controller" filename="libgazebo_ros_laser.so">
+            <topicName>${prefix_topic}/scan</topicName>
+            <frameName>/${prefix}_link</frameName>
+          </plugin>
+        </sensor>
       </xacro:unless>
-      <sensor type="${ray_type}" name="${prefix}_sensor">
-        <pose>0 0 0 0 0 0</pose>
-        <visualize>false</visualize>
-        <update_rate>30</update_rate>
-        <ray>
-          <scan>
-            <horizontal>
-              <samples>1081</samples>
-              <resolution>1</resolution>
-              <min_angle>${min_angle}</min_angle>
-              <max_angle>${max_angle}</max_angle>
-            </horizontal>
-          </scan>
-          <range>
-            <min>0.10</min>
-            <max>30.0</max>
-            <resolution>0.01</resolution>
-          </range>
-          <noise>
-            <type>gaussian</type>
-            <mean>0.0</mean>
-            <stddev>0.001</stddev>
-          </noise>
-        </ray>
-        <plugin name="${prefix}_controller" filename="${plugin_lib}">
-          <topicName>${prefix_topic}/scan</topicName>
-          <frameName>/${prefix}_link</frameName>
-        </plugin>
-      </sensor>
     </gazebo>
   </xacro:macro>
